File: PCB/2020-08-18 Motor Board.sch (EAGLE design)
At the start: 21 parts

Commit message: updates schematics, dimensions and placement.
Parts:
- removed CB-UC-1, CB-UC-2: 100n, Passives:C-M2012
- removed IC-COM-1: MODULE-RS485-3MM5-JACK-X2, 2020-08-18 Motor Board:MODULE-RS485-3MM5-JACK-X2
- removed IC-UC-1: LONGAN-NANO, 2020-08-18 Motor Board:LONGAN-NANO
- removed LF-UC-1: BEAD 500mA, Passives:L-M2012
- removed RL-HB-2, RL-HB-3: 2.2K, Passives:R-M2012
- added CB-ADC-1, CB-ADC-2, CB-ENC-1, CB-ENC-2, CB-PWR-2, CB-PWR1: 100n, Passives:C-M2012
- added CF-ADC-1: 10n, Passives:C-M2012
- added CP-PWR-1: C+-TH3.5-8.0, Passives:C+-TH3.5-8.0
- added DP-ENC-1, DP-ENC-2: BAT54S-SOT23, 2020-08-18 Motor Board:BAT54S-SOT23
- added F-ENC-1: 500mA, Passives:PTC-M2012
- added IC-ADC-1: MCP6282-SO8, 2020-08-18 Motor Board:MCP6282-SO8
- added IC-ENC-1: LM393-SO8, 2020-08-18 Motor Board:LM393-SO8
- added JP-ENC-1: (no value), 2020-08-18 Motor Board:PINHD-1X3
- added LD-ENC-1, LD-ENC-2, LD-ENC-3: GREEN, Passives:LED-M2012
- added LF-ADC-1, LF-ADC-2, LF-ENC-1, LF-ENC2, LF-PWR-1, LF-PWR2: BEAD 500mA, Passives:L-M2012
- added RF-ENC-1, RF-ENC-2, RL-ADC-1, RL-ENC-1, RL-ENC-2, RL-ENC-3, RL-PWR-1, RU-ENC-3, RU-PWR-1: 2.2K, Passives:R-M2012
- added RS-ENC-1, RS-ENC-2, RS-ENC-3, RU-ENC-1, RU-ENC-2: 330, Passives:R-M2012
- added RS-UC-1, RS-UC-2: RX4-M2012-X4, Passives:RX4-M2012-X4
- added U$3: MODULE-LONGAN-NANO, 2020-08-18 Motor Board:MODULE-LONGAN-NANO
- renumbered CB-PWR-1 to CB-PWR-3, CB-UC-3 to CF-PWR-1, LD_HB_BW to LD-HB-BW
Connections:
- removed net N$10: IC-HB-1.SENSE_EN
- removed net N$17: CON-ENC-1.3
- removed net N$18: CON-ENC-1.4
- removed net N$6: IC-HB-1.INA
- removed net N$7: IC-HB-1.INB
- removed net N$8: IC-HB-1.SEL0
- removed net UC-HB-INA-SEL0: IC-UC-1.PB8_TIMER32__I2C0SCL_CAN0RX
- new net ENC-BIAS: IC-ENC-1A.-IN, IC-ENC-1B.-IN, RL-ENC-3.1, RU-ENC-3.2
- new net ENC-CHA: CON-ENC-1.3, DP-ENC-1.C1A2, RL-ENC-1.1, RU-ENC-1.1
- new net ENC-CHB: CON-ENC-1.4, DP-ENC-2.C1A2, RL-ENC-2.1, RU-ENC-2.1
- new net HB-INA: IC-HB-1.INA, RS-UC-1.2B
- new net HB-INB: IC-HB-1.INB, RS-UC-1.4B
- new net HB-MSENSE-EN: IC-HB-1.SENSE_EN, RS-UC-2.2B
- new net HB-PWM: IC-HB-1.PWM, RS-UC-1.1B
- new net HB-SEL0: IC-HB-1.SEL0, RS-UC-1.3B
- new net HB-SEL1: IC-HB-1.SEL1, RS-UC-2.1B
- new net HB-SENSE: IC-ADC-1A.+IN, IC-HB-1.SENSE, RL-ADC-1.1
- new net N$12: LD-ENC-1.-, RS-ENC-1.1
- new net N$13: CB-PWR-2.2, LF-PWR-1.2, MOD-PWR-1.IN
- new net N$14: CB-ENC-1.2, F-ENC-1.2, LF-ENC-1.1
- new net N$15: LD-ENC-3.-, RS-ENC-3.1
- new net N$16: RS-UC-2.4A
- new net N$19: RS-UC-2.3B
- new net N$4: IC-ENC-1A.+IN, RF-ENC-1.1, RL-ENC-1.2
- new net PWR-SENSE-VIN: CF-ADC-1.1, IC-ADC-1B.+IN, RL-PWR-1.1, RU-PWR-1.2
- new net UC-HB-INA: RS-UC-1.2A, U$3.B8_TIMER32__I2C0SCL_CAN0RX
- new net UC-HB-SEL0: RS-UC-1.3A, U$3.B7_TIMER31_I2C0SDA__UART0RXI
- new net UC-PWR-SENSE-IIN: IC-PWR-1.SENSE, U$3.A6_ADC06_SPI0MISO_TIMER20__TIMER0BRKIN
- new net VENC#+: F-ENC-1.1, JP-ENC-1.2
- net MOT+: now also IC-HB-1.OUT-A; no longer IC-HB-1.OUT-B
- net MOT-: now also IC-HB-1.OUT-B; no longer IC-HB-1.OUT-A
- net N$11: now also IC-ENC-1B.+IN, RF-ENC-2.1, RL-ENC-2.2; no longer IC-HB-1.SENSE
- net N$20: now also RS-UC-2.4B; no longer IC-PWR-1.SENSE
- net N$5: now also LD-ENC-2.-, RS-ENC-2.1; no longer IC-HB-1.PWM
- net N$9: now also RS-UC-2.3A; no longer IC-HB-1.SEL1
- net UC-COM-RXE#: now also U$3.B13_UART2CTS_TIMER00ON_SPI1SCK_I2S1CLK_CAN1TX; no longer IC-COM-1.RXEN#, IC-UC-1.PB13_UART2CTS_TIMER00ON_SPI1SCK_I2S1CLK_CAN1TX
- net UC-COM-RXI: now also U$3.B11_UART2RXI_I2C1SDA__TIMER13; no longer IC-COM-1.RXO, IC-UC-1.PB11_UART2RXI_I2C1SDA__TIMER13
- net UC-COM-TXE: now also U$3.B12_UART2CLK_TIMER0BRKIN_SPI1NSS_I2S1WS_I2C1SMBA_CAN1RX; no longer IC-COM-1.TXEN, IC-UC-1.PB12_UART2CLK_TIMER0BRKIN_SPI1NSS_I2S1WS_I2C1SMBA_CAN1RX
- net UC-COM-TXO: now also U$3.B10_UART2TXO_I2C1SCL__TIMER12; no longer IC-COM-1.TXI, IC-UC-1.PB10_UART2TXO_I2C1SCL__TIMER12
- net UC-ENC-CHA: now also IC-ENC-1A.OUT, LD-ENC-1.+, RF-ENC-1.2, U$3.B4_JTAG0NJTRST_SPI2MISO__SPI0MISO_TIMER20; no longer IC-UC-1.PB4_JTAG0NJTRST_SPI2MISO__SPI0MISO_TIMER20
- net UC-ENC-CHB: now also IC-ENC-1B.OUT, LD-ENC-2.+, RF-ENC-2.2, U$3.B5_I2C0SMBA_SPI2MOSI_I2S2SD__CAN1RX_SPI0MOSI_TIMER21; no longer IC-UC-1.PB5_I2C0SMBA_SPI2MOSI_I2S2SD__CAN1RX_SPI0MOSI_TIMER21
- net UC-HB-INB: now also RS-UC-1.4A, U$3.B9_TIMER33__I2C0SDA_CAN0TX; no longer IC-UC-1.PB9_TIMER33__I2C0SDA_CAN0TX
- net UC-HB-MSENSE-EN: now also RS-UC-2.2A, U$3.B15_TIMER02ON_SPI1MOSI_I2S1SD; no longer IC-UC-1.PA3_ADC03_TIMER13_TIMER43_UART1RXI
- net UC-HB-PWM: now also RS-UC-1.1A, U$3.B6_TIMER30_I2C0SCL__UART0TXO_CAN1TX; no longer IC-UC-1.PB6_TIMER30_I2C0SCL__UART0TXO_CAN1TX
- net UC-HB-SEL1: now also RS-UC-2.1A, U$3.B14_UART2RTS_TIMER01ON_SPI1MISO; no longer IC-UC-1.PB7_TIMER31_I2C0SDA__UART0RXI
- net UC-HB-SENSE-IOUT: now also IC-ADC-1A.-IN, IC-ADC-1A.OUT, U$3.A0_ADC00_TIMER10ETI_TIMER40_UART1CTS_WKUP; no longer IC-UC-1.PA0_ADC00_TIMER10ETI_TIMER40_UART1CTS_WKUP
- net UC-PWR-SENSE-VIN: now also IC-ADC-1B.-IN, IC-ADC-1B.OUT, U$3.A4_ADC04_UART1CLK_DAC0_SPI0NSS__SPI2NSS_I2S2WS; no longer IC-UC-1.PA4_ADC04_UART1CLK_DAC0_SPI0NSS__SPI2NSS_I2S2WS, RL-HB-2.2, RL-HB-3.1
- net VADC+: now also CB-ADC-2.2, CF-PWR-1.1, IC-ADC-1P.V+, LF-ADC-1.2; no longer CB-UC-2.2, LF-UC-1.2
- net VADC-: now also CB-ADC-2.1, CB-PWR-3.2, IC-ADC-1P.V-, IC-PWR-1.-, LF-ADC-2.2, RL-ADC-1.2; no longer CB-UC-1.1, CB-UC-2.1
- net VENC+: now also CB-ENC-2.2, DP-ENC-1.C2, DP-ENC-2.C2, IC-ENC-1P.V+, LD-ENC-3.+, LF-ENC-1.2, RU-ENC-1.2, RU-ENC-2.2, RU-ENC-3.1
- net VENC-: now also CB-ENC-2.1, DP-ENC-1.A1, DP-ENC-2.A1, IC-ENC-1P.V-, LF-ENC2.2, RL-ENC-3.2
- net VIN#+: now also CB-PWR1.2, CP-PWR-1.+, LF-PWR-1.1, RU-PWR-1.1; no longer MOD-PWR-1.IN, RL-HB-2.1
- net VIN+: now also JP-ENC-1.1
- net VIN-: now also CB-PWR1.1, CP-PWR-1.-, LF-PWR2.1; no longer MOD-PWR-1.COM
- net VUC+: now also CB-ADC-1.2, CP-UC-1.+, JP-ENC-1.3, LF-ADC-1.1, U$3.5V; no longer CB-UC-1.2, IC-COM-1.5V0, IC-UC-1.5V0, LF-UC-1.1
- net VUC-: now also CB-ADC-1.1, CB-ENC-1.1, CB-PWR-2.1, CF-ADC-1.2, CP-UC-1.-, LF-ADC-2.1, LF-ENC2.1, LF-PWR2.2, MOD-PWR-1.COM, RL-PWR-1.2, RS-ENC-1.2, RS-ENC-2.2, RS-ENC-3.2, U$3.0V; no longer CB-PWR-3.2, CF-PWR-1.1, IC-COM-1.0V0, IC-PWR-1.-, IC-UC-1.0V, RL-HB-3.2
Other:
- note added: "Sense VIN"
- note added: "Threshold Comparator"
- note removed: "RS485"
- note removed: "Transceiver Module"
- moved on the sheet: CON-ENC-1, CP-UC-1, MOD-PWR-1
